File: PCB/PMA-183PLN+/PMA-183PLN+.kicad_pcb (KiCad board)
At the start: 4 copper layers, 35 x 35 mm, 25 parts, among them U1 PMA-183PLN+, U2 MIC5219-2.6YM5-TR

Commit message: Included pcb libraries in repository under '_dependencies' with projects linked to them using relative paths
Parts:
-  : footprint FabDrawingTemplates:FabDrawing-4Layer-Metric-Compact-OSH -> rf-dfs:FabDrawing-4Layer-Metric-Compact-OSH
-  : footprint footprints.pretty:GCPW_osh3_90mm_user -> rf-dfs:GCPW_osh3_90mm_user
- 2.6VDC, GND, Vin: footprint TestPoint:TestPoint_Loop_D2.54mm_Drill1.5mm_Beaded -> rf-dfs:TestPoint_Loop_D2.54mm_Drill1.5mm_Beaded
- C1, C2, C3, C4, C5, C6, C7, C8: footprint Capacitor_SMD:C_0402_1005Metric -> rf-dfs:C_0402_1005Metric
- C9: footprint Capacitor_SMD:C_1206_3216Metric -> rf-dfs:C_1206_3216Metric
- G***: footprint footprints.pretty:nrao1_6mm_silk -> rf-dfs:nrao1_6mm_silk
- R1, R2: footprint Resistor_SMD:R_0603_1608Metric -> rf-dfs:R_0603_1608Metric
- REF** (x4): footprint MountingHole:MountingHole_2.7mm_M2.5 -> rf-dfs:MountingHole_2.7mm_M2.5
- RF-In, RF-Out: footprint footprints:Mueller BU-1420761881 -> rf-dfs:Mueller BU-1420761881
- U1: footprint Mini-Circuits:QFN51P250X350X85-17N -> rf-dfs:QFN51P250X350X85-17N
- U2: footprint imports:SOT-23-5_M5_MCH -> rf-dfs:SOT-23-5_M5_MCH
Changed lines of the file:
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@@
       (layer "B.Paste" (type "Bottom Solder Paste"))
       (layer "B.SilkS" (type "Bottom Silk Screen") (color "White") (material "Liquid Photo"))
-      (copper_finish "ENIG")
+      (copper_finish "None")
       (dielectric_constraints yes)
     )
@@
   (net 7 "Net-(IC2-VE)")
   (net 8 "Net-(IC2-VDD)")
-  (footprint "Resistor_SMD:R_0603_1608Metric" (layer "F.Cu")
+  (footprint "rf-dfs:R_0603_1608Metric" (layer "F.Cu")
     (at 140.2 82.065 90)
     (descr "Resistor SMD 0603 (1608 Metric), square (rectangular) end terminal, IPC_7351 nominal, (Body size source: IPC-SM-782 page 72, https://www.pcb-3d.com/wordpress/wp-content/uploads/ipc-sm-782a_amendment_1_and_2.pdf), generated with kicad-footprint-generator")
@@
     )
   )
-  (footprint "Capacitor_SMD:C_0402_1005Metric" (layer "F.Cu")
+  (footprint "rf-dfs:C_0402_1005Metric" (layer "F.Cu")
     (at 140.68 88.13)
     (descr "Capacitor SMD 0402 (1005 Metric), square (rectangular) end terminal, IPC_7351 nominal, (Body size source: IPC-SM-782 page 76, https://www.pcb-3d.com/wordpress/wp-content/uploads/ipc-sm-782a_amendment_1_and_2.pdf), generated with kicad-footprint-generator")
@@
     )
   )
-  (footprint "Capacitor_SMD:C_1206_3216Metric" (layer "F.Cu")
+  (footprint "rf-dfs:C_1206_3216Metric" (layer "F.Cu")
     (at 144.325 79.4)
     (descr "Capacitor SMD 1206 (3216 Metric), square (rectangular) end terminal, IPC_7351 nominal, (Body size source: IPC-SM-782 page 76, https://www.pcb-3d.com/wordpress/wp-content/uploads/ipc-sm-782a_amendment_1_and_2.pdf), generated with kicad-footprint-generator")
@@
     )
   )
-  (footprint "Capacitor_SMD:C_0402_1005Metric" (layer "F.Cu")
+  (footprint "rf-dfs:C_0402_1005Metric" (layer "F.Cu")
     (at 131.7 76.86 -90)
     (descr "Capacitor SMD 0402 (1005 Metric), square (rectangular) end terminal, IPC_7351 nominal, (Body size source: IPC-SM-782 page 76, https://www.pcb-3d.com/wordpress/wp-content/uploads/ipc-sm-782a_amendment_1_and_2.pdf), generated with kicad-footprint-generator")
@@
     )
   )
-  (footprint "Capacitor_SMD:C_0402_1005Metric" (layer "F.Cu")
+  (footprint "rf-dfs:C_0402_1005Metric" (layer "F.Cu")
     (at 140.68 90.1)
     (descr "Capacitor SMD 0402 (1005 Metric), square (rectangular) end terminal, IPC_7351 nominal, (Body size source: IPC-SM-782 page 76, https://www.pcb-3d.com/wordpress/wp-content/uploads/ipc-sm-782a_amendment_1_and_2.pdf), generated with kicad-footprint-generator")
@@
     )
   )
-  (footprint "Capacitor_SMD:C_0402_1005Metric" (layer "F.Cu")
+  (footprint "rf-dfs:C_0402_1005Metric" (layer "F.Cu")
     (at 137.92 86.16)
     (descr "Capacitor SMD 0402 (1005 Metric), square (rectangular) end terminal, IPC_7351 nominal, (Body size source: IPC-SM-782 page 76, https://www.pcb-3d.com/wordpress/wp-content/uploads/ipc-sm-782a_amendment_1_and_2.pdf), generated with kicad-footprint-generator")
@@
     )
   )
-  (footprint "TestPoint:TestPoint_Loop_D2.54mm_Drill1.5mm_Beaded" (layer "F.Cu")
+  (footprint "rf-dfs:TestPoint_Loop_D2.54mm_Drill1.5mm_Beaded" (layer "F.Cu")
     (at 128.8 86.32)
     (descr "wire loop with bead as test point, loop diameter2.548mm, hole diameter 1.5mm")
@@
     )
   )
-  (footprint "Capacitor_SMD:C_0402_1005Metric" (layer "F.Cu")
+  (footprint "rf-dfs:C_0402_1005Metric" (layer "F.Cu")
     (at 140.2 77.59 -90)
     (descr "Capacitor SMD 0402 (1005 Metric), square (rectangular) end terminal, IPC_7351 nominal, (Body size source: IPC-SM-782 page 76, https://www.pcb-3d.com/wordpress/wp-content/uploads/ipc-sm-782a_amendment_1_and_2.pdf), generated with kicad-footprint-generator")
@@
     )
   )
-  (footprint "footprints:Mueller BU-1420761881" (layer "F.Cu")
+  (footprint "rf-dfs:Mueller BU-1420761881" (layer "F.Cu")
     (at 149.31 94 180)
     (descr "Molex SMA RF Connectors, Edge Mount, (http://www.molex.com/pdm_docs/sd/732511150_sd.pdf)")
@@
     )
   )
-  (footprint "imports:SOT-23-5_M5_MCH" (layer "F.Cu")
+  (footprint "rf-dfs:SOT-23-5_M5_MCH" (layer "F.Cu")
     (at 137 76.16)
     (tags "MIC5219-2.6YM5-TR ")
@@
     )
   )
-  (footprint "FabDrawingTemplates:FabDrawing-4Layer-Metric-Compact-OSH" (layer "F.Cu")
+  (footprint "rf-dfs:FabDrawing-4Layer-Metric-Compact-OSH" (layer "F.Cu")
     (at 55.5 135.5)
     (attr through_hole)
@@
       (stroke (width 0.1) (type solid)) (fill solid) (layer "Dwgs.User"))
   )
-  (footprint "TestPoint:TestPoint_Loop_D2.54mm_Drill1.5mm_Beaded" (layer "F.Cu")
+  (footprint "rf-dfs:TestPoint_Loop_D2.54mm_Drill1.5mm_Beaded" (layer "F.Cu")
     (at 128.8 81.24)
     (descr "wire loop with bead as test point, loop diameter2.548mm, hole diameter 1.5mm")
@@
     )
   )
-  (footprint "Mini-Circuits:QFN51P250X350X85-17N" (layer "F.Cu")
+  (footprint "rf-dfs:QFN51P250X350X85-17N" (layer "F.Cu")
     (at 139.3 94 -90)
     (descr "JV2579-DFN=16_")
@@
     )
   )
-  (footprint "MountingHole:MountingHole_2.7mm_M2.5" (layer "F.Cu")
+  (footprint "rf-dfs:MountingHole_2.7mm_M2.5" (layer "F.Cu")
     (at 150.85 103.15)
     (descr "Mounting Hole 2.7mm, no annular, M2.5")
@@
     (pad "" np_thru_hole circle (at 0 0) (size 2.7 2.7) (drill 2.7) (layers "*.Mask" "F.Cu" "In1.Cu" "In2.Cu" "B.Cu"))
   )
-  (footprint "Resistor_SMD:R_0603_1608Metric" (layer "F.Cu")
+  (footprint "rf-dfs:R_0603_1608Metric" (layer "F.Cu")
     (at 139.3 84.5)
     (descr "Resistor SMD 0603 (1608 Metric), square (rectangular) end terminal, IPC_7351 nominal, (Body size source: IPC-SM-782 page 72, https://www.pcb-3d.com/wordpress/wp-content/uploads/ipc-sm-782a_amendment_1_and_2.pdf), generated with kicad-footprint-generator")
@@
     )
   )
-  (footprint "TestPoint:TestPoint_Loop_D2.54mm_Drill1.5mm_Beaded" (layer "F.Cu")
+  (footprint "rf-dfs:TestPoint_Loop_D2.54mm_Drill1.5mm_Beaded" (layer "F.Cu")
     (at 128.8 76.16)
     (descr "wire loop with bead as test point, loop diameter2.548mm, hole diameter 1.5mm")
@@
     )
   )
-  (footprint "Capacitor_SMD:C_0402_1005Metric" (layer "F.Cu")
+  (footprint "rf-dfs:C_0402_1005Metric" (layer "F.Cu")
     (at 137.92 90.1)
     (descr "Capacitor SMD 0402 (1005 Metric), square (rectangular) end terminal, IPC_7351 nominal, (Body size source: IPC-SM-782 page 76, https://www.pcb-3d.com/wordpress/wp-content/uploads/ipc-sm-782a_amendment_1_and_2.pdf), generated with kicad-footprint-generator")
@@
     )
   )
-  (footprint "footprints.pretty:nrao1_6mm_silk" (layer "F.Cu")
+  (footprint "rf-dfs:nrao1_6mm_silk" (layer "F.Cu")
     (at 129.2 101.5)
     (attr board_only exclude_from_pos_files exclude_from_bom)
@@
       (stroke (width 0) (type solid)) (fill solid) (layer "F.SilkS"))
   )
-  (footprint "MountingHole:MountingHole_2.7mm_M2.5" (layer "F.Cu")
+  (footprint "rf-dfs:MountingHole_2.7mm_M2.5" (layer "F.Cu")
     (at 150.85 74.15)
     (descr "Mounting Hole 2.7mm, no annular, M2.5")
@@
     (pad "" np_thru_hole circle (at 0 0) (size 2.7 2.7) (drill 2.7) (layers "*.Mask" "F.Cu" "In1.Cu" "In2.Cu" "B.Cu"))
   )
-  (footprint "MountingHole:MountingHole_2.7mm_M2.5" (layer "F.Cu")
+  (footprint "rf-dfs:MountingHole_2.7mm_M2.5" (layer "F.Cu")
     (at 121.85 74.15)
     (descr "Mounting Hole 2.7mm, no annular, M2.5")
@@
     (pad "" np_thru_hole circle (at 0 0) (size 2.7 2.7) (drill 2.7) (layers "*.Mask" "F.Cu" "In1.Cu" "In2.Cu" "B.Cu"))
   )
-  (footprint "footprints:Mueller BU-1420761881" (layer "F.Cu")
+  (footprint "rf-dfs:Mueller BU-1420761881" (layer "F.Cu")
     (at 123.39 94)
     (descr "Molex SMA RF Connectors, Edge Mount, (http://www.molex.com/pdm_docs/sd/732511150_sd.pdf)")
@@
     )
   )
-  (footprint "Capacitor_SMD:C_0402_1005Metric" (layer "F.Cu")
+  (footprint "rf-dfs:C_0402_1005Metric" (layer "F.Cu")
     (at 137.92 88.13)
     (descr "Capacitor SMD 0402 (1005 Metric), square (rectangular) end terminal, IPC_7351 nominal, (Body size source: IPC-SM-782 page 76, https://www.pcb-3d.com/wordpress/wp-content/uploads/ipc-sm-782a_amendment_1_and_2.pdf), generated with kicad-footprint-generator")
@@
     )
   )
-  (footprint "MountingHole:MountingHole_2.7mm_M2.5" (layer "F.Cu")
+  (footprint "rf-dfs:MountingHole_2.7mm_M2.5" (layer "F.Cu")
     (at 121.85 103.15)
     (descr "Mounting Hole 2.7mm, no annular, M2.5")
@@
     (pad "" np_thru_hole circle (at 0 0) (size 2.7 2.7) (drill 2.7) (layers "*.Cu" "*.Mask"))
   )
-  (footprint "Capacitor_SMD:C_0402_1005Metric" (layer "F.Cu")
+  (footprint "rf-dfs:C_0402_1005Metric" (layer "F.Cu")
     (at 140.68 86.16)
     (descr "Capacitor SMD 0402 (1005 Metric), square (rectangular) end terminal, IPC_7351 nominal, (Body size source: IPC-SM-782 page 76, https://www.pcb-3d.com/wordpress/wp-content/uploads/ipc-sm-782a_amendment_1_and_2.pdf), generated with kicad-footprint-generator")
@@
     )
   )
-  (footprint "footprints.pretty:GCPW_osh3_90mm_user" (layer "F.Cu")
+  (footprint "rf-dfs:GCPW_osh3_90mm_user" (layer "F.Cu")
     (at 207 147.5)
     (attr board_only exclude_from_pos_files exclude_from_bom)
