File: PCB/PMA-183PLN+/PMA-183PLN+.kicad_sch (KiCad schematic)
At the start: 18 parts, among them J1 Conn_Coaxial, J2 Conn_Coaxial, U1 PMA-183PLN+, U2 MIC5219-2.6YM5-TR

Commit message: Included pcb libraries in repository under '_dependencies' with projects linked to them using relative paths
Parts:
- C1, C2, C3, C4, C5, C6, C7, C8: symbol Device:C_Small -> rf-dfs:C_Small
- C9: symbol Device:C_Polarized_Small -> rf-dfs:C_Polarized_Small
- J1, J2: symbol Connector:Conn_Coaxial -> rf-dfs:Conn_Coaxial
- R1, R2: symbol Device:R_Small_US -> rf-dfs:R_Small_US
- TP1, TP2, TP3: symbol Connector:TestPoint -> rf-dfs:TestPoint
- U1: symbol PMA-183PLN+:PMA-183PLN+ -> rf-dfs:PMA-183PLN+
- U2: symbol MIC5219-2.6YM5:MIC5219-2.6YM5-TR -> rf-dfs:MIC5219-2.6YM5-TR
Changed lines of the file:
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@@
     )
   )
-  (symbol (lib_id "Connector:TestPoint") (at 81.28 45.72 0) (unit 1)
+  (symbol (lib_id "rf-dfs:TestPoint") (at 81.28 45.72 0) (unit 1)
     (in_bom yes) (on_board yes) (dnp no) (fields_autoplaced)
     (property "Reference" "TP1" (at 83.82 41.148 0)
@@
     )
   )
-  (symbol (lib_id "MIC5219-2.6YM5:MIC5219-2.6YM5-TR") (at 125.73 45.72 0) (unit 1)
+  (symbol (lib_id "rf-dfs:MIC5219-2.6YM5-TR") (at 125.73 45.72 0) (unit 1)
     (in_bom yes) (on_board yes) (dnp no) (fields_autoplaced)
     (property "Reference" "U2" (at 153.67 35.56 0)
@@
     )
   )
-  (symbol (lib_id "Device:C_Small") (at 184.15 95.25 180) (unit 1)
+  (symbol (lib_id "rf-dfs:C_Small") (at 184.15 95.25 180) (unit 1)
     (in_bom yes) (on_board yes) (dnp no) (fields_autoplaced)
     (property "Reference" "C3" (at 186.69 93.9736 0)
@@
     )
   )
-  (symbol (lib_id "Connector:TestPoint") (at 184.15 45.72 0) (mirror y) (unit 1)
+  (symbol (lib_id "rf-dfs:TestPoint") (at 184.15 45.72 0) (mirror y) (unit 1)
     (in_bom yes) (on_board yes) (dnp no)
     (property "Reference" "TP3" (at 181.61 41.148 0)
@@
     )
   )
-  (symbol (lib_id "Device:C_Small") (at 119.38 99.06 270) (unit 1)
+  (symbol (lib_id "rf-dfs:C_Small") (at 119.38 99.06 270) (unit 1)
     (in_bom yes) (on_board yes) (dnp no) (fields_autoplaced)
     (property "Reference" "C6" (at 119.3736 92.71 90)
@@
     )
   )
-  (symbol (lib_id "Device:C_Small") (at 102.87 49.53 0) (unit 1)
+  (symbol (lib_id "rf-dfs:C_Small") (at 102.87 49.53 0) (unit 1)
     (in_bom yes) (on_board yes) (dnp no) (fields_autoplaced)
     (property "Reference" "C7" (at 105.41 48.2663 0)
@@
     )
   )
-  (symbol (lib_id "Device:C_Small") (at 158.75 95.25 180) (unit 1)
+  (symbol (lib_id "rf-dfs:C_Small") (at 158.75 95.25 180) (unit 1)
     (in_bom yes) (on_board yes) (dnp no) (fields_autoplaced)
     (property "Reference" "C1" (at 161.29 93.9736 0)
@@
     )
   )
-  (symbol (lib_id "Connector:Conn_Coaxial") (at 81.28 124.46 0) (mirror y) (unit 1)
+  (symbol (lib_id "rf-dfs:Conn_Coaxial") (at 81.28 124.46 0) (mirror y) (unit 1)
     (in_bom yes) (on_board yes) (dnp no)
     (property "Reference" "J1" (at 77.47 123.4832 0)
@@
     )
   )
-  (symbol (lib_id "Device:C_Small") (at 209.55 58.42 0) (unit 1)
+  (symbol (lib_id "rf-dfs:C_Small") (at 209.55 58.42 0) (unit 1)
     (in_bom yes) (on_board yes) (dnp no) (fields_autoplaced)
     (property "Reference" "C8" (at 212.09 57.1563 0)
@@
     )
   )
-  (symbol (lib_id "Device:C_Polarized_Small") (at 196.85 58.42 0) (unit 1)
+  (symbol (lib_id "rf-dfs:C_Polarized_Small") (at 196.85 58.42 0) (unit 1)
     (in_bom yes) (on_board yes) (dnp no) (fields_autoplaced)
     (property "Reference" "C9" (at 199.39 56.6039 0)
@@
     )
   )
-  (symbol (lib_id "Device:C_Small") (at 171.45 95.25 180) (unit 1)
+  (symbol (lib_id "rf-dfs:C_Small") (at 171.45 95.25 180) (unit 1)
     (in_bom yes) (on_board yes) (dnp no) (fields_autoplaced)
     (property "Reference" "C2" (at 173.99 93.9736 0)
@@
     )
   )
-  (symbol (lib_id "Device:C_Small") (at 119.38 78.74 270) (unit 1)
+  (symbol (lib_id "rf-dfs:C_Small") (at 119.38 78.74 270) (unit 1)
     (in_bom yes) (on_board yes) (dnp no) (fields_autoplaced)
     (property "Reference" "C4" (at 119.3736 72.39 90)
@@
     )
   )
-  (symbol (lib_id "Connector:TestPoint") (at 102.87 45.72 0) (unit 1)
+  (symbol (lib_id "rf-dfs:TestPoint") (at 102.87 45.72 0) (unit 1)
     (in_bom yes) (on_board yes) (dnp no) (fields_autoplaced)
     (property "Reference" "TP2" (at 105.41 41.148 0)
@@
     )
   )
-  (symbol (lib_id "PMA-183PLN+:PMA-183PLN+") (at 151.13 111.76 270) (unit 1)
+  (symbol (lib_id "rf-dfs:PMA-183PLN+") (at 151.13 111.76 270) (unit 1)
     (in_bom yes) (on_board yes) (dnp no) (fields_autoplaced)
     (property "Reference" "U1" (at 119.38 115.4683 90)
@@
     )
   )
-  (symbol (lib_id "Device:R_Small_US") (at 146.05 88.9 90) (unit 1)
+  (symbol (lib_id "rf-dfs:R_Small_US") (at 146.05 88.9 90) (unit 1)
     (in_bom yes) (on_board yes) (dnp no) (fields_autoplaced)
     (property "Reference" "R2" (at 146.05 82.55 90)
@@
     )
   )
-  (symbol (lib_id "Device:R_Small_US") (at 184.15 77.47 180) (unit 1)
+  (symbol (lib_id "rf-dfs:R_Small_US") (at 184.15 77.47 180) (unit 1)
     (in_bom yes) (on_board yes) (dnp no) (fields_autoplaced)
     (property "Reference" "R1" (at 186.69 76.2 0)
@@
     )
   )
-  (symbol (lib_id "Device:C_Small") (at 119.38 88.9 270) (unit 1)
+  (symbol (lib_id "rf-dfs:C_Small") (at 119.38 88.9 270) (unit 1)
     (in_bom yes) (on_board yes) (dnp no) (fields_autoplaced)
     (property "Reference" "C5" (at 119.3736 82.55 90)
@@
     )
   )
-  (symbol (lib_id "Connector:Conn_Coaxial") (at 209.55 127 0) (unit 1)
+  (symbol (lib_id "rf-dfs:Conn_Coaxial") (at 209.55 127 0) (unit 1)
     (in_bom yes) (on_board yes) (dnp no)
     (property "Reference" "J2" (at 213.36 126.0232 0)
