File: PCB/PMA2-63LN+/002.35.20.15.20-001-PCB-Biasing.kicad_sch (KiCad schematic)
At the start: 9 parts

Commit message: Included pcb libraries in repository under '_dependencies' with projects linked to them using relative paths
Parts:
- C? (x4): symbol Device:C_Small -> rf-dfs:C_Small
- L?: symbol Device:L -> rf-dfs:L
- R? (x2): symbol Device:R -> rf-dfs:R
- TP1: symbol Connector:TestPoint -> rf-dfs:TestPoint
- U?: symbol PMA2-63LN+:PMA2-63LN+ -> rf-dfs:PMA2-63LN+_1
Changed lines of the file:
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@@
     )
   )
-  (symbol (lib_id "Device:C_Small") (at 190.5 83.82 90) (unit 1)
+  (symbol (lib_id "rf-dfs:C_Small") (at 190.5 83.82 90) (unit 1)
     (in_bom yes) (on_board yes) (dnp no) (fields_autoplaced)
     (property "Reference" "C?" (at 190.5063 77.47 90)
@@
     )
   )
-  (symbol (lib_id "Device:L") (at 181.61 105.41 0) (unit 1)
+  (symbol (lib_id "rf-dfs:L") (at 181.61 105.41 0) (unit 1)
     (in_bom yes) (on_board yes) (dnp no) (fields_autoplaced)
     (property "Reference" "L?" (at 182.88 104.14 0)
@@
     )
   )
-  (symbol (lib_id "Device:C_Small") (at 190.5 97.79 90) (unit 1)
+  (symbol (lib_id "rf-dfs:C_Small") (at 190.5 97.79 90) (unit 1)
     (in_bom yes) (on_board yes) (dnp no) (fields_autoplaced)
     (property "Reference" "C?" (at 190.5063 91.44 90)
@@
     )
   )
-  (symbol (lib_name "PMA2-63LN+_1") (lib_id "PMA2-63LN+:PMA2-63LN+") (at 124.46 105.41 0) (unit 1)
+  (symbol (lib_name "PMA2-63LN+_1") (lib_id "rf-dfs:PMA2-63LN+_1") (at 124.46 105.41 0) (unit 1)
     (in_bom yes) (on_board yes) (dnp no) (fields_autoplaced)
     (property "Reference" "U?" (at 147.32 95.25 0)
@@
     )
   )
-  (symbol (lib_id "Device:C_Small") (at 190.5 113.03 90) (unit 1)
+  (symbol (lib_id "rf-dfs:C_Small") (at 190.5 113.03 90) (unit 1)
     (in_bom yes) (on_board yes) (dnp no) (fields_autoplaced)
     (property "Reference" "C?" (at 190.5063 106.68 90)
@@
     )
   )
-  (symbol (lib_id "Device:C_Small") (at 111.76 110.49 90) (unit 1)
+  (symbol (lib_id "rf-dfs:C_Small") (at 111.76 110.49 90) (unit 1)
     (in_bom yes) (on_board yes) (dnp no) (fields_autoplaced)
     (property "Reference" "C?" (at 111.7663 104.14 90)
@@
     )
   )
-  (symbol (lib_id "Connector:TestPoint") (at 121.92 82.55 0) (unit 1)
+  (symbol (lib_id "rf-dfs:TestPoint") (at 121.92 82.55 0) (unit 1)
     (in_bom yes) (on_board yes) (dnp no) (fields_autoplaced)
     (property "Reference" "TP1" (at 124.46 77.978 0)
@@
     )
   )
-  (symbol (lib_id "Device:R") (at 116.84 92.71 90) (unit 1)
+  (symbol (lib_id "rf-dfs:R") (at 116.84 92.71 90) (unit 1)
     (in_bom yes) (on_board yes) (dnp yes) (fields_autoplaced)
     (property "Reference" "R?" (at 116.84 86.36 90)
@@
     )
   )
-  (symbol (lib_id "Device:R") (at 127 92.71 90) (unit 1)
+  (symbol (lib_id "rf-dfs:R") (at 127 92.71 90) (unit 1)
     (in_bom yes) (on_board yes) (dnp yes) (fields_autoplaced)
     (property "Reference" "R?" (at 127 86.36 90)
