File: PCB/PMA2-63LN+/002.35.20.15.20-001-PCB-LNA.kicad_sch (KiCad schematic)
At the start: 12 parts, among them J1 Conn_Coaxial, J2 Conn_Coaxial, J3 Conn_Coaxial, U3 YAT-1A+, U4 L7805, U5 L7805

Commit message: Included pcb libraries in repository under '_dependencies' with projects linked to them using relative paths
Parts:
- C10, C11, C12, C9: symbol Device:C_Small -> rf-dfs:C_Small
- J1, J2, J3: symbol Connector:Conn_Coaxial -> rf-dfs:Conn_Coaxial
- TP1: symbol Connector:TestPoint -> rf-dfs:TestPoint
- U3: symbol YAT-1A+:YAT-1A+ -> rf-dfs:YAT-1A+
- U4, U5: symbol Regulator_Linear:L7805 -> rf-dfs:L7805
Changed lines of the file:
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@@
     )
   )
-  (symbol (lib_id "Device:C_Small") (at 242.57 50.8 0) (unit 1)
+  (symbol (lib_id "rf-dfs:C_Small") (at 242.57 50.8 0) (unit 1)
     (in_bom yes) (on_board yes) (dnp no) (fields_autoplaced)
     (property "Reference" "C12" (at 245.11 49.5363 0)
@@
     )
   )
-  (symbol (lib_id "Connector:TestPoint") (at 48.26 50.8 90) (unit 1)
+  (symbol (lib_id "rf-dfs:TestPoint") (at 48.26 50.8 90) (unit 1)
     (in_bom yes) (on_board yes) (dnp no) (fields_autoplaced)
     (property "Reference" "TP1" (at 44.958 45.72 90)
@@
     )
   )
-  (symbol (lib_id "Regulator_Linear:L7805") (at 223.52 45.72 0) (unit 1)
+  (symbol (lib_id "rf-dfs:L7805") (at 223.52 45.72 0) (unit 1)
     (in_bom yes) (on_board yes) (dnp no) (fields_autoplaced)
     (property "Reference" "U5" (at 223.52 39.37 0)
@@
     )
   )
-  (symbol (lib_id "Connector:Conn_Coaxial") (at 69.85 45.72 0) (mirror y) (unit 1)
+  (symbol (lib_id "rf-dfs:Conn_Coaxial") (at 69.85 45.72 0) (mirror y) (unit 1)
     (in_bom yes) (on_board yes) (dnp no)
     (property "Reference" "J3" (at 66.04 44.7432 0)
@@
     )
   )
-  (symbol (lib_id "Regulator_Linear:L7805") (at 152.4 45.72 0) (unit 1)
+  (symbol (lib_id "rf-dfs:L7805") (at 152.4 45.72 0) (unit 1)
     (in_bom yes) (on_board yes) (dnp no) (fields_autoplaced)
     (property "Reference" "U4" (at 152.4 39.37 0)
@@
     )
   )
-  (symbol (lib_id "Device:C_Small") (at 200.66 50.8 0) (unit 1)
+  (symbol (lib_id "rf-dfs:C_Small") (at 200.66 50.8 0) (unit 1)
     (in_bom yes) (on_board yes) (dnp no) (fields_autoplaced)
     (property "Reference" "C11" (at 203.2 49.5363 0)
@@
     )
   )
-  (symbol (lib_id "Device:C_Small") (at 171.45 50.8 0) (unit 1)
+  (symbol (lib_id "rf-dfs:C_Small") (at 171.45 50.8 0) (unit 1)
     (in_bom yes) (on_board yes) (dnp no) (fields_autoplaced)
     (property "Reference" "C10" (at 173.99 49.5363 0)
@@
     )
   )
-  (symbol (lib_id "Device:C_Small") (at 129.54 50.8 0) (unit 1)
+  (symbol (lib_id "rf-dfs:C_Small") (at 129.54 50.8 0) (unit 1)
     (in_bom yes) (on_board yes) (dnp no) (fields_autoplaced)
     (property "Reference" "C9" (at 132.08 49.5363 0)
@@
     )
   )
-  (symbol (lib_id "YAT-1A+:YAT-1A+") (at 124.46 121.92 0) (unit 1)
+  (symbol (lib_id "rf-dfs:YAT-1A+") (at 124.46 121.92 0) (unit 1)
     (in_bom yes) (on_board yes) (dnp no) (fields_autoplaced)
     (property "Reference" "U3" (at 147.32 111.76 0)
@@
     )
   )
-  (symbol (lib_id "Connector:Conn_Coaxial") (at 60.96 124.46 0) (mirror y) (unit 1)
+  (symbol (lib_id "rf-dfs:Conn_Coaxial") (at 60.96 124.46 0) (mirror y) (unit 1)
     (in_bom yes) (on_board yes) (dnp no) (fields_autoplaced)
     (property "Reference" "J1" (at 61.2774 118.11 0)
@@
     )
   )
-  (symbol (lib_id "Connector:Conn_Coaxial") (at 245.11 127 0) (unit 1)
+  (symbol (lib_id "rf-dfs:Conn_Coaxial") (at 245.11 127 0) (unit 1)
     (in_bom yes) (on_board yes) (dnp no) (fields_autoplaced)
     (property "Reference" "J2" (at 244.7926 120.65 0)
@@
     )
   )
-  (symbol (lib_id "Connector:TestPoint") (at 81.28 45.72 0) (unit 1)
+  (symbol (lib_id "rf-dfs:TestPoint") (at 81.28 45.72 0) (unit 1)
     (in_bom yes) (on_board yes) (dnp no) (fields_autoplaced)
     (property "Reference" "TP1" (at 83.82 41.148 0)
