File: PCB/TSS-183A+/TSS-183A+.kicad_sch (KiCad schematic)
At the start: 18 parts, among them J1 Conn_Coaxial, J2 Conn_Coaxial, U1 TSS-183A+, U2 L7805

Commit message: Included pcb libraries in repository under '_dependencies' with projects linked to them using relative paths
Parts:
- C1, C2, C3, C4, C5, C6, C7, C8: symbol Device:C_Small -> rf-dfs:C_Small
- J1, J2: symbol Connector:Conn_Coaxial -> rf-dfs:Conn_Coaxial
- L1, L2: symbol Device:L_Small -> rf-dfs:L_Small
- TP1, TP2, TP3, TP4: symbol Connector:TestPoint -> rf-dfs:TestPoint
- U1: symbol TSS-183A+:TSS-183A+ -> rf-dfs:TSS-183A+
- U2: symbol Regulator_Linear:L7805 -> rf-dfs:L7805
Changed lines of the file:
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@@
     )
   )
-  (symbol (lib_id "Connector:TestPoint") (at 81.28 45.72 0) (unit 1)
+  (symbol (lib_id "rf-dfs:TestPoint") (at 81.28 45.72 0) (unit 1)
     (in_bom yes) (on_board yes) (dnp no) (fields_autoplaced)
     (property "Reference" "TP1" (at 83.82 41.148 0)
@@
     )
   )
-  (symbol (lib_id "Device:C_Small") (at 161.29 81.28 0) (unit 1)
+  (symbol (lib_id "rf-dfs:C_Small") (at 161.29 81.28 0) (unit 1)
     (in_bom yes) (on_board yes) (dnp no) (fields_autoplaced)
     (property "Reference" "C2" (at 163.83 80.0163 0)
@@
     )
   )
-  (symbol (lib_id "Regulator_Linear:L7805") (at 146.05 45.72 0) (unit 1)
+  (symbol (lib_id "rf-dfs:L7805") (at 146.05 45.72 0) (unit 1)
     (in_bom yes) (on_board yes) (dnp no) (fields_autoplaced)
     (property "Reference" "U2" (at 146.05 39.37 0)
@@
     )
   )
-  (symbol (lib_id "Connector:TestPoint") (at 184.15 45.72 0) (mirror y) (unit 1)
+  (symbol (lib_id "rf-dfs:TestPoint") (at 184.15 45.72 0) (mirror y) (unit 1)
     (in_bom yes) (on_board yes) (dnp no)
     (property "Reference" "TP3" (at 181.61 41.148 0)
@@
     )
   )
-  (symbol (lib_id "Device:C_Small") (at 102.87 49.53 0) (unit 1)
+  (symbol (lib_id "rf-dfs:C_Small") (at 102.87 49.53 0) (unit 1)
     (in_bom yes) (on_board yes) (dnp no) (fields_autoplaced)
     (property "Reference" "C8" (at 105.41 48.2663 0)
@@
     )
   )
-  (symbol (lib_id "Device:C_Small") (at 121.92 148.59 0) (unit 1)
+  (symbol (lib_id "rf-dfs:C_Small") (at 121.92 148.59 0) (unit 1)
     (in_bom yes) (on_board yes) (dnp no) (fields_autoplaced)
     (property "Reference" "C5" (at 124.46 147.3263 0)
@@
     )
   )
-  (symbol (lib_id "Connector:TestPoint") (at 146.05 156.21 180) (unit 1)
+  (symbol (lib_id "rf-dfs:TestPoint") (at 146.05 156.21 180) (unit 1)
     (in_bom yes) (on_board yes) (dnp no) (fields_autoplaced)
     (property "Reference" "TP4" (at 148.59 158.242 0)
@@
     )
   )
-  (symbol (lib_id "Connector:Conn_Coaxial") (at 81.28 124.46 0) (mirror y) (unit 1)
+  (symbol (lib_id "rf-dfs:Conn_Coaxial") (at 81.28 124.46 0) (mirror y) (unit 1)
     (in_bom yes) (on_board yes) (dnp no)
     (property "Reference" "J1" (at 77.47 123.4832 0)
@@
     )
   )
-  (symbol (lib_id "Device:C_Small") (at 161.29 97.79 90) (unit 1)
+  (symbol (lib_id "rf-dfs:C_Small") (at 161.29 97.79 90) (unit 1)
     (in_bom yes) (on_board yes) (dnp no) (fields_autoplaced)
     (property "Reference" "C3" (at 161.2963 91.44 90)
@@
     )
   )
-  (symbol (lib_id "Device:C_Small") (at 165.1 49.53 0) (unit 1)
+  (symbol (lib_id "rf-dfs:C_Small") (at 165.1 49.53 0) (unit 1)
     (in_bom yes) (on_board yes) (dnp no) (fields_autoplaced)
     (property "Reference" "C7" (at 167.64 48.2663 0)
@@
     )
   )
-  (symbol (lib_id "Device:C_Small") (at 162.56 148.59 180) (unit 1)
+  (symbol (lib_id "rf-dfs:C_Small") (at 162.56 148.59 180) (unit 1)
     (in_bom yes) (on_board yes) (dnp no) (fields_autoplaced)
     (property "Reference" "C4" (at 165.1 147.3136 0)
@@
     )
   )
-  (symbol (lib_id "Device:C_Small") (at 173.99 81.28 0) (unit 1)
+  (symbol (lib_id "rf-dfs:C_Small") (at 173.99 81.28 0) (unit 1)
     (in_bom yes) (on_board yes) (dnp no) (fields_autoplaced)
     (property "Reference" "C1" (at 176.53 80.0163 0)
@@
     )
   )
-  (symbol (lib_id "Connector:TestPoint") (at 102.87 45.72 0) (unit 1)
+  (symbol (lib_id "rf-dfs:TestPoint") (at 102.87 45.72 0) (unit 1)
     (in_bom yes) (on_board yes) (dnp no) (fields_autoplaced)
     (property "Reference" "TP2" (at 105.41 41.148 0)
@@
     )
   )
-  (symbol (lib_id "Device:L_Small") (at 143.51 148.59 0) (mirror y) (unit 1)
+  (symbol (lib_id "rf-dfs:L_Small") (at 143.51 148.59 0) (mirror y) (unit 1)
     (in_bom yes) (on_board yes) (dnp no)
     (property "Reference" "L2" (at 142.24 147.32 0)
@@
     )
   )
-  (symbol (lib_id "Device:C_Small") (at 130.81 97.79 90) (unit 1)
+  (symbol (lib_id "rf-dfs:C_Small") (at 130.81 97.79 90) (unit 1)
     (in_bom yes) (on_board yes) (dnp no) (fields_autoplaced)
     (property "Reference" "C6" (at 130.8163 91.44 90)
@@
     )
   )
-  (symbol (lib_id "Device:L_Small") (at 146.05 91.44 0) (mirror y) (unit 1)
+  (symbol (lib_id "rf-dfs:L_Small") (at 146.05 91.44 0) (mirror y) (unit 1)
     (in_bom yes) (on_board yes) (dnp no)
     (property "Reference" "L1" (at 144.78 90.17 0)
@@
     )
   )
-  (symbol (lib_id "Connector:Conn_Coaxial") (at 209.55 124.46 0) (unit 1)
+  (symbol (lib_id "rf-dfs:Conn_Coaxial") (at 209.55 124.46 0) (unit 1)
     (in_bom yes) (on_board yes) (dnp no)
     (property "Reference" "J2" (at 213.36 123.4832 0)
@@
     )
   )
-  (symbol (lib_id "TSS-183A+:TSS-183A+") (at 128.27 121.92 0) (unit 1)
+  (symbol (lib_id "rf-dfs:TSS-183A+") (at 128.27 121.92 0) (unit 1)
     (in_bom yes) (on_board yes) (dnp no) (fields_autoplaced)
     (property "Reference" "U1" (at 166.37 115.4683 0)
