File: PCB/PMA3-14LN+/PMA3-14LN+.kicad_sch (KiCad schematic)
At the start: 19 parts, among them J1 Conn_Coaxial, J2 Conn_Coaxial, U1 PMA3-14LN+, U2 L7806

Commit message: Included pcb libraries in repository under '_dependencies' with projects linked to them using relative paths
Parts:
- C1, C2, C3, C4, C5, C6, C7, C8, C9: symbol Device:C_Small -> rf-dfs:C_Small
- J1, J2: symbol Connector:Conn_Coaxial -> rf-dfs:Conn_Coaxial
- L1, L2: symbol Device:L_Small -> rf-dfs:L_Small
- R1: symbol Device:R_Small_US -> rf-dfs:R_Small_US
- TP1, TP2, TP3: symbol Connector:TestPoint -> rf-dfs:TestPoint
- U1: symbol PMA3-14LN+:PMA3-14LN+ -> rf-dfs:PMA3-14LN+
- U2: symbol Regulator_Linear:L7806 -> rf-dfs:L7806
Changed lines of the file:
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@@
     )
   )
-  (symbol (lib_id "Connector:TestPoint") (at 88.9 45.72 0) (unit 1)
+  (symbol (lib_id "rf-dfs:TestPoint") (at 88.9 45.72 0) (unit 1)
     (in_bom yes) (on_board yes) (dnp no) (fields_autoplaced)
     (property "Reference" "TP1" (at 91.44 41.148 0)
@@
     )
   )
-  (symbol (lib_id "Device:C_Small") (at 97.79 124.46 90) (unit 1)
+  (symbol (lib_id "rf-dfs:C_Small") (at 97.79 124.46 90) (unit 1)
     (in_bom yes) (on_board yes) (dnp no) (fields_autoplaced)
     (property "Reference" "C1" (at 97.7963 118.11 90)
@@
     )
   )
-  (symbol (lib_id "Device:C_Small") (at 97.79 101.6 90) (unit 1)
+  (symbol (lib_id "rf-dfs:C_Small") (at 97.79 101.6 90) (unit 1)
     (in_bom yes) (on_board yes) (dnp no) (fields_autoplaced)
     (property "Reference" "C5" (at 97.7963 95.25 90)
@@
     )
   )
-  (symbol (lib_id "Device:C_Small") (at 184.15 130.81 180) (unit 1)
+  (symbol (lib_id "rf-dfs:C_Small") (at 184.15 130.81 180) (unit 1)
     (in_bom yes) (on_board yes) (dnp no) (fields_autoplaced)
     (property "Reference" "C4" (at 186.69 129.5336 0)
@@
     )
   )
-  (symbol (lib_id "Connector:TestPoint") (at 184.15 45.72 0) (mirror y) (unit 1)
+  (symbol (lib_id "rf-dfs:TestPoint") (at 184.15 45.72 0) (mirror y) (unit 1)
     (in_bom yes) (on_board yes) (dnp no)
     (property "Reference" "TP3" (at 181.61 41.148 0)
@@
     )
   )
-  (symbol (lib_id "Device:C_Small") (at 194.31 101.6 90) (unit 1)
+  (symbol (lib_id "rf-dfs:C_Small") (at 194.31 101.6 90) (unit 1)
     (in_bom yes) (on_board yes) (dnp no) (fields_autoplaced)
     (property "Reference" "C6" (at 194.3163 95.25 90)
@@
     )
   )
-  (symbol (lib_id "Device:C_Small") (at 121.92 49.53 0) (unit 1)
+  (symbol (lib_id "rf-dfs:C_Small") (at 121.92 49.53 0) (unit 1)
     (in_bom yes) (on_board yes) (dnp no) (fields_autoplaced)
     (property "Reference" "C9" (at 124.46 48.2663 0)
@@
     )
   )
-  (symbol (lib_id "Device:C_Small") (at 194.31 88.9 90) (unit 1)
+  (symbol (lib_id "rf-dfs:C_Small") (at 194.31 88.9 90) (unit 1)
     (in_bom yes) (on_board yes) (dnp no) (fields_autoplaced)
     (property "Reference" "C8" (at 194.3163 82.4919 90)
@@
     )
   )
-  (symbol (lib_id "Regulator_Linear:L7806") (at 143.51 45.72 0) (unit 1)
+  (symbol (lib_id "rf-dfs:L7806") (at 143.51 45.72 0) (unit 1)
     (in_bom yes) (on_board yes) (dnp no) (fields_autoplaced)
     (property "Reference" "U2" (at 143.51 39.37 0)
@@
     )
   )
-  (symbol (lib_id "Connector:Conn_Coaxial") (at 81.28 124.46 0) (mirror y) (unit 1)
+  (symbol (lib_id "rf-dfs:Conn_Coaxial") (at 81.28 124.46 0) (mirror y) (unit 1)
     (in_bom yes) (on_board yes) (dnp no)
     (property "Reference" "J1" (at 77.47 123.4832 0)
@@
     )
   )
-  (symbol (lib_id "Device:C_Small") (at 107.95 130.81 180) (unit 1)
+  (symbol (lib_id "rf-dfs:C_Small") (at 107.95 130.81 180) (unit 1)
     (in_bom yes) (on_board yes) (dnp no) (fields_autoplaced)
     (property "Reference" "C3" (at 110.49 129.5336 0)
@@
     )
   )
-  (symbol (lib_id "PMA3-14LN+:PMA3-14LN+") (at 120.65 121.92 0) (unit 1)
+  (symbol (lib_id "rf-dfs:PMA3-14LN+") (at 120.65 121.92 0) (unit 1)
     (in_bom yes) (on_board yes) (dnp no)
     (property "Reference" "U1" (at 173.99 115.4683 0)
@@
     )
   )
-  (symbol (lib_id "Device:L_Small") (at 184.15 113.03 0) (unit 1)
+  (symbol (lib_id "rf-dfs:L_Small") (at 184.15 113.03 0) (unit 1)
     (in_bom yes) (on_board yes) (dnp no) (fields_autoplaced)
     (property "Reference" "L2" (at 185.42 111.76 0)
@@
     )
   )
-  (symbol (lib_id "Device:C_Small") (at 194.31 124.46 90) (unit 1)
+  (symbol (lib_id "rf-dfs:C_Small") (at 194.31 124.46 90) (unit 1)
     (in_bom yes) (on_board yes) (dnp no) (fields_autoplaced)
     (property "Reference" "C2" (at 194.3163 118.11 90)
@@
     )
   )
-  (symbol (lib_id "Device:L_Small") (at 107.95 113.03 0) (unit 1)
+  (symbol (lib_id "rf-dfs:L_Small") (at 107.95 113.03 0) (unit 1)
     (in_bom yes) (on_board yes) (dnp no) (fields_autoplaced)
     (property "Reference" "L1" (at 109.22 111.76 0)
@@
     )
   )
-  (symbol (lib_id "Connector:TestPoint") (at 121.92 45.72 0) (unit 1)
+  (symbol (lib_id "rf-dfs:TestPoint") (at 121.92 45.72 0) (unit 1)
     (in_bom yes) (on_board yes) (dnp no) (fields_autoplaced)
     (property "Reference" "TP2" (at 124.46 41.148 0)
@@
     )
   )
-  (symbol (lib_id "Device:R_Small_US") (at 132.08 88.9 90) (unit 1)
+  (symbol (lib_id "rf-dfs:R_Small_US") (at 132.08 88.9 90) (unit 1)
     (in_bom yes) (on_board yes) (dnp no) (fields_autoplaced)
     (property "Reference" "R1" (at 132.08 82.55 90)
@@
     )
   )
-  (symbol (lib_id "Device:C_Small") (at 97.79 88.9 90) (unit 1)
+  (symbol (lib_id "rf-dfs:C_Small") (at 97.79 88.9 90) (unit 1)
     (in_bom yes) (on_board yes) (dnp no) (fields_autoplaced)
     (property "Reference" "C7" (at 97.7963 82.55 90)
@@
     )
   )
-  (symbol (lib_id "Connector:Conn_Coaxial") (at 209.55 124.46 0) (unit 1)
+  (symbol (lib_id "rf-dfs:Conn_Coaxial") (at 209.55 124.46 0) (unit 1)
     (in_bom yes) (on_board yes) (dnp no)
     (property "Reference" "J2" (at 213.36 123.4832 0)

Commit message: PMA3-14LN+ Rev B Complete
Parts:
- J1, J2: footprint footprints:SMA_Molex_73251-1153_EdgeMount_Horizontal_TunedOSH -> rf-dfs:Mueller BU-1420761881-RevB
Changed lines of the file:
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@@
       (effects (font (size 1.27 1.27)) (justify left))
     )
-    (property "Footprint" "footprints:SMA_Molex_73251-1153_EdgeMount_Horizontal_TunedOSH" (at 81.28 124.46 0)
+    (property "Footprint" "rf-dfs:Mueller BU-1420761881-RevB" (at 81.28 124.46 0)
       (effects (font (size 1.27 1.27)) hide)
     )
@@
       (effects (font (size 1.27 1.27)) (justify left))
     )
-    (property "Footprint" "footprints:SMA_Molex_73251-1153_EdgeMount_Horizontal_TunedOSH" (at 209.55 124.46 0)
-      (effects (font (size 1.27 1.27)) hide)
-    )
+    (property "Footprint" "rf-dfs:Mueller BU-1420761881-RevB" (at 209.55 124.46 0)
+      (effects (font (size 1.27 1.27)) hide)
+    )
